File: PCB/WIP/SensorStick.brd (EAGLE design)
At the start: 74.9 x 39.4 mm, 73 parts, among them U1 TPD4F003DQDR, U2 BMI088, U3 BMI088, U4 BMI088, U5 STM32H743ZIT6, U6 STM32H743ZIT6, U7 STM32H743ZIT6, U8 STM32H743ZIT6, Y1 ECS-TXO-3225MV-400-TR

Commit message: preliminary PCB design with main 3 sensors on board, still a lot of small details to figure out
Parts:
- added C28, C29, C30, C31, C32, C33: (no value), capacitor-wima:C2.5-4
- added FL1, FL3: BLM03AG601SN1D, BLM03AG601SN1D:BEADC0603X33N
- added U10, U11, U9: LIS3MDLTR, LIS3MDLTR:XDCR_LIS3MDLTR
- moved R9 430.2 mm to (-61.0, -411.0), turned to 0 degrees
- moved R8 425.8 mm to (-61.0, -407.7)
- moved JP7 420.0 mm to (-58.2, -403.4)
- moved U3 390.1 mm to (-58.9, -455.7)
- moved U2 381.7 mm to (-58.9, -438.9)
- moved U1 358.2 mm to (-42.2, -343.2), turned to 0 degrees
- moved U4 296.3 mm to (-58.9, -369.1)
- moved R10 277.4 mm to (-61.0, -469.9)
- moved IC2 218.8 mm to (-44.5, -421.9)
- moved C25 52.8 mm to (-59.9, -376.9)
- moved FL2 52.8 mm to (-61.2, -380.2)
- moved C24 51.1 mm to (-52.6, -368.6)
- moved C27 44.5 mm to (-54.9, -376.9)
Connections:
- removed net 3V1: IC2.1, IC2.2
- removed net GNDA: U2.4, U3.4
- removed net GNDIO: U2.6, U3.6
- removed net I2C2_SDA1: BAROMETER.3, R2.1
- removed net I2C2_SDA2: BAROMETER1.3, R12.1
- removed net I2C2_SDA3: BAROMETER2.3, R15.1
- removed net N$4: IC2.24
- removed net N$7: IC2.23
- removed net VDDIO: U2.11, U3.11
- new net 3V4: C24.1, C25.1, FL2.2, U4.3
- new net 3V5: C31.1, C32.1, FL3.2, U3.3
- new net CSB_ACCEL2: U3.14
- new net CSB_ACCEL3: U2.14
- new net CSB_GYRO2: U3.5
- new net CSB_GYRO3: U2.5
- new net N$10: C33.1, FL3.1, U3.11
- new net N$9: C30.1, FL1.1, U2.11
- new net NRST1: U1.4
- new net SWCLK_O1: JP7.3
- new net SWDIO_O1: JP7.5
- new net SWO_O1: JP7.1
- net 3V2: now also C28.1, C29.1, FL1.2, U2.3; no longer C24.1, C25.1, FL2.2, U4.3
- net 3V3: now also IC2.1, IC2.2, L2.2, L3.2, L7.2, U10.5, U10.6, U11.5, U11.6, U9.5, U9.6; no longer L2.1, L3.1, L7.1
- net EXTI0: now also U2.16, U3.16
- net EXTI2: now also U2.12, U3.12
- net GND: now also C28.2, C29.2, C30.2, C31.2, C32.2, C33.2, U10.3, U11.3, U2.4, U2.6, U2.7, U3.4, U3.6, U3.7, U9.3
- net GPIO_EXTI0: now also U6.114
- net GPIO_EXTI1: now also U6.115
- net GPIO_EXTI2: now also U6.116
- net GPIO_EXTI3: now also U6.117
- net GPIO_EXTI4: now also U6.118
- net I2C1_SCL: now also BAROMETER.4, R1.1
- net I2C1_SDA: now also BAROMETER.3, R2.1
- net I2C2_SCL: no longer BAROMETER.4, BAROMETER2.4, R1.1, R13.1
- net I2C2_SDA: now also BAROMETER1.3, R12.1
- net I2C3_SCL: now also BAROMETER2.4, R13.1
- net I2C3_SDA: now also BAROMETER2.3, R15.1
- net IMU_INT2: now also U2.1, U3.1
- net IMU_INT4: now also U2.13, U3.13
- net N$2: now also L3.1; no longer L3.2
- net N$3: now also L2.1; no longer L2.2
- net N$6: now also L7.1; no longer L7.2
- net NRST: no longer U1.4
- net SPI2_MISO: now also U3.10, U3.15
- net SPI2_MOSI: now also U3.9
- net SPI2_SCK: now also U3.8
- net SPI3_MISO: now also U2.10, U2.15
- net SPI3_MOSI: now also U2.9
- net SPI3_SCK: now also U2.8
- net SPI4_CS: now also U9.10
- net SPI4_MISO: now also U9.11
- net SPI4_MOSI: now also U9.9
- net SPI4_SCK: now also U9.1
- net SPI5_CS: now also U11.10
- net SPI5_MISO: now also U11.11
- net SPI5_MOSI: now also U11.9
- net SPI5_SCK: now also U11.1
- net SPI6_CS: now also U10.10
- net SPI6_MISO: now also U10.11
- net SPI6_MOSI: now also U10.9
- net SPI6_SCK: now also U10.1
- net SWCLK_O: no longer JP7.3
- net SWDIO_O: no longer JP7.5
- net SWO_O: no longer JP7.1
- net VDD: no longer U2.3, U3.3
Routing:
- net I2C1_SDA: track 42.0 -> 0.00 mm, vias 2 -> 0
- net I2C1_SCL: track 40.1 -> 0.00 mm, vias 2 -> 0
- net USART1_TX: track 16.8 -> 0.00 mm, vias 2 -> 0
- net USART1_RX: track 14.3 -> 0.00 mm, vias 2 -> 0
- net SWDIO: track 11.9 -> 0.00 mm, vias 2 -> 0
- net SWO_O: track 9.21 -> 0.00 mm
- net SWCLK_O: track 6.84 -> 0.00 mm
- net SWO: track 6.03 -> 0.00 mm
- net SWCLK: track 4.75 -> 0.00 mm
- net NRST_O: track 2.84 -> 0.00 mm
- net 3V3: track 50.1 -> 47.4 mm, vias 13 -> 11
- net SWDIO_O: track 2.46 -> 0.00 mm
- net GND: track 71.4 -> 69.6 mm, vias 21 -> 20
- net NRST: track 75.9 -> 75.1 mm
