File: PCB/WIP/SensorStick.sch (EAGLE design)
At the start: 88 parts, among them U1 TPD4F003DQDR, U10 LIS3MDLTR, U11 LIS3MDLTR, U2 BMI088, U3 BMI088, U4 BMI088, U5 STM32H743ZIT6, U9 LIS3MDLTR, Y1 ECS-TXO-3225MV-400-TR

Commit message: slight changes but this is rough draft 1 officially
Parts:
- removed R10, R22, R25: 0, SparkFun-Resistors:0OHM-0603-1/10W-5%
Connections:
- removed net IMU_INT1: R22.1, U3.INT2
- removed net IMU_INT2: R10.2, U4.INT2
- removed net IMU_INT4: R10.1, U4.INT4
- removed net IMU_INT5: R25.1, U2.INT2
- removed net IMU_INT6: R25.2, U2.INT4
- removed net JTDI: U5G$1.PA15(JTDI)
- removed net LPUART1_RX: U5G$1.PA10
- removed net LPUART1_TX: U5G$1.PA9
- removed net N$18: RC.4
- removed net N$21: LIDAR.5
- removed net N$22: LIDAR.4
- removed net SPI2_CS: U5G$2.PB12
- removed net SPI3_CS: U5G$1.PA4
- removed net UART4_RX: U5G$1.PA1
- removed net UART4_TX: U5G$1.PA0
- removed net UART8_RX: U5G$3.PE0
- removed net UART8_TX: U5G$3.PE1
- new net GPIO1: LIDAR.4, U5G$4.PG1
- new net N$20: U4.INT2, U4.INT4
- new net N$23: U2.INT2, U2.INT4
- new net XSHUT: LIDAR.5, U5G$2.PC1
- net GND: no longer RC.6
- net IMU_INT3: now also U3.INT2; no longer R22.2
- net N$19: now also RC.6; no longer RC.5

Commit message: cleaned up layout
Parts:
- removed L1: BLM03AG601SN1D, BLM03AG601SN1D:BLM03AG601SN1D
- removed SV1: (no value), con-lsta:FE05-1
- added C38, C39: 1.0uF, SparkFun-Capacitors:1.0UF-0805-25V-10%
- added CON1: B4B-ZR, jst:B4B-ZR
- added GPS: (no value), con-lsta:FE05-1
- added JP1: (no value), pinhead:PINHD-2X3
- added RADIO: B6B-ZR, jst:B6B-ZR
- C14: value 0.1uF -> 1.0uF; device SparkFun-Capacitors:0.1UF-0603-25V-5% -> SparkFun-Capacitors:1.0UF-0805-25V-10%
Connections:
- new net DM: CON1.2
- new net DP: CON1.3
- new net GND1: C14.2, C15.2, C16.2, C17.2, C18.2, C20.2, C21.2, C22.2
- new net GND2: C19.2
- new net GND3: C38.2
- new net GND4: C39.2
- new net UART4_RX: JP1.4, U5G$1.PA11
- new net UART4_TX: JP1.2, U5G$1.PA12
- new net UART8_RX: RADIO.3, U5G$3.PE0
- new net UART8_TX: RADIO.2, U5G$3.PE1
- new net VREF1: C14.1
- new net VREF2: C19.1
- new net VREF3: C38.1
- new net VREF4: C39.1
- net 3V3: now also GPS.5, RADIO.1; no longer C15.1, C16.1, C17.1, C18.1, C20.1, C21.1, C22.1, L1.2, SV1.5
- net 5V_IN: now also CON1.4
- net GND: now also CON1.1, GPS.4; no longer C14.2, C15.2, C16.2, C17.2, C18.2, C19.1, C20.2, C21.2, C22.2, SV1.4
- net GPIO_EXTI1: now also GPS.1; no longer SV1.1
- net N$19: now also RADIO.6
- net NRST_O: now also JP1.6
- net SWCLK_O: now also JP1.3
- net SWDIO_O: now also JP1.5
- net SWO_O: now also JP1.1
- net USART2_RX: now also GPS.3; no longer SV1.3
- net USART2_TX: now also GPS.2; no longer SV1.2
- net VREF: now also C15.1, C16.1, C17.1, C18.1, C20.1, C21.1, C22.1; no longer C14.1, C19.2, L1.1
Other:
- note added: "Barometer"
- note added: "Buttons"
- note added: "Bypass Capacitors"
- note added: "IMUs"
- note added: "Magnetometers"
- note added: "Off-board components"
- note added: "Power Module"
- note added: "Reset"
- note added: "STM32H743"
- note added: "User"
- moved on the sheet: BAROMETER, BAROMETER1, BAROMETER2, C1, C10, C11, C12, C13, C14, C15, C16, C17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

Commit message: bypass cap fixes and other minor stuffs
Parts:
- removed CON1: B4B-ZR, jst:B4B-ZR
- removed U11, U9: LIS3MDLTR, LIS3MDLTR:LIS3MDLTR
- added C40, C49: 1.0uF, SparkFun-Capacitors:1.0UF-0805-25V-10%
- added C41, C42, C43, C44, C45, C46, C47, C48: 0.1uF, SparkFun-Capacitors:0.1UF-0603-25V-5%
- added C50: 0.1uf, SparkFun-Capacitors:1.0UF-0805-25V-10%
- added C51, C52: 5.6pF, SparkFun-Capacitors:1.0UF-0805-25V-10%
- added J1: 10118192-0001LF, ce-capstone:10118192-0001LF
- added R10: 220, ce-capstone:RT0402FRE07220RL
- added U6, U7: LIS3MDLTR, LIS3MDLTR:LIS3MDLTR
- added Y2: ABLS-8.000MHZ-B2-T, ce-capstone:ABLS-8.000MHZ-B2-T
- C3: value 0.1uF -> 2.2uF; device SparkFun-Capacitors:0.1UF-0603-25V-5% -> SparkFun-Capacitors:1.0UF-0805-25V-10%
- C34: value 0.1uF -> 1.0uF; device SparkFun-Capacitors:0.1UF-0603-25V-5% -> SparkFun-Capacitors:1.0UF-0805-25V-10%
- C35: value 0.1uF -> 0.1uf; device SparkFun-Capacitors:0.1UF-0603-25V-5% -> SparkFun-Capacitors:1.0UF-0805-25V-10%
- C37: value 1.0uF -> 2.2uf
Connections:
- removed net DM: CON1.2
- removed net DP: CON1.3
- removed net N$11: C36.2, U10.C1
- removed net N$12: C37.1, U5G$1.VCAP
- removed net N$4: C34.2, U9.C1
- removed net VREF: C15.1, C16.1, C17.1, C18.1, C20.1, C21.1, C22.1, U5G$1.VREF+
- new net AGND: C3.1, C34.1, C35.1, C37.1, C49.1, C50.1
- new net OSC_OUT: R10.1, U5G$1.PH1/OSC_OUT
- new net VBAT: C40.2, U5G$1.VBAT
- new net VCAP: C3.2, C37.2, U5G$1.VCAP
- new net VDD: C15.1, C16.1, C17.1, C18.1, C20.1, C21.1, C22.1
- new net VDDA: C34.2, C35.2, U5G$1.VDDA
- new net VREFP: C49.2, C50.2, U5G$1.VREF+
- net 3V3: now also C36.2, C41.2, C42.2, C43.2, C44.2, C45.2, C46.2, C47.2, C48.2, U6.VDD, U6.VDD_IO, U7.VDD, U7.VDD_IO; no longer C3.2, U11.VDD, U11.VDD_IO, U5G$1.VBAT, U5G$1.VDDA, U9.VDD, U9.VDD_IO
- net 5V_IN: now also J1.VUSB; no longer CON1.4
- net GND: now also C40.1, C41.1, C42.1, C43.1, C44.1, C45.1, C46.1, C47.1, C48.1, C51.1, C52.1, J1.GND, U10.C1, U6.C1, U6.GND, U6.RSVD1, U6.RSVD2, U7.C1, U7.GND, U7.RSVD1, U7.RSVD2; no longer C3.1, C34.1, C35.1, C37.2, CON1.1, U11.GND, U11.RSVD1, U11.RSVD2, U9.GND, U9.RSVD1, U9.RSVD2
- net N$7: now also C52.2, R10.2, Y2.1; no longer C35.2, U11.C1
- net OSC_IN: now also C51.2, U5G$1.PH0/OSC_IN, Y2.2
- net SPI4_CS: now also U7.CS; no longer U9.CS
- net SPI4_MISO: now also U7.SDA/SDI/SDO; no longer U9.SDA/SDI/SDO
- net SPI4_MOSI: now also U7.SDO/SA1; no longer U9.SDO/SA1
- net SPI4_SCK: now also U7.SCL/SPC; no longer U9.SCL/SPC
- net SPI5_CS: now also U6.CS; no longer U11.CS
- net SPI5_MISO: now also U6.SDA/SDI/SDO; no longer U11.SDA/SDI/SDO
- net SPI5_MOSI: now also U6.SDO/SA1; no longer U11.SDO/SA1
- net SPI5_SCK: now also U6.SCL/SPC; no longer U11.SCL/SPC
Other:
- moved on the sheet: C14, C15, C16, C17, C18, C19, C20, C21, C22, C3, C34, C35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
