File: PCB/WIP/RedundantSensors.brd (EAGLE design)
At the start: 99 x 98.7 mm, 121 parts, among them J1 10118192-0001LF, U1 TPD4F003DQDR, U10 LIS3MDLTR, U2 BMI088, U3 BMI088, U4 BMI088, U5 STM32H743ZIT6, U6 LIS3MDLTR, U7 LIS3MDLTR, Y1 8MHz, Y2 8MHz

Commit message: snapshot before making changes suggested by phil
Parts:
- removed JP1: (no value), pinhead:2X03
- removed LIDAR, OP_FLOW, RADIO, RC: B6B-ZR, jst:B6B-ZR
- added J2, J4: JST-SH-4_SMT_V, con-JST-SH:BM04B-SRSS-TB
- added J3: 503182-1852, 503182-1852:MOLEX_503182-1852
- added JP5: (no value), jumper:JP5Q
- added R31: 10k, SparkFun-Resistors:0603
- added R32, R33: 1000, SparkFun-Resistors:0402
- added X1: LiDAR, con-jst2:6FLZ-SM
- added X3: RC, con-jst:6FLZ-SM
- Y1: value 8MHz -> 32MHz
- moved U6 50.2 mm to (7.62, 68.6)
- moved JP2 49.5 mm to (6.35, 39.4)
- moved R16 47.6 mm to (85.1, 39.4)
- moved U7 28.0 mm to (30.5, 30.5)
- moved R19 16.5 mm to (41.9, 34.3), turned to 0 degrees
- moved U$1 15.7 mm to (6.35, 17.8)
- moved R8 12.5 mm to (49.5, 35.6), turned to 0 degrees
- moved C55 10.5 mm to (33.0, 58.4)
- moved C56 10.5 mm to (33.0, 54.6)
- moved L2 10.5 mm to (22.9, 78.7)
- moved C4 10.5 mm to (22.9, 76.2)
- moved BAROMETER1 10.5 mm to (19.1, 77.5)
- moved R12 10.5 mm to (17.8, 72.4)
- moved C11 10.5 mm to (20.3, 80.0)
- moved C12 10.5 mm to (11.4, 80.0)
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Connections:
- removed net IMU_INT3: U3.1, U3.13
- removed net N$20: U4.1, U4.13
- removed net N$23: U2.1, U2.13
- new net 3.3V: JP5.7, JP5.8
- new net DRDY1: U10.8, U5.125
- new net DRDY2: U5.44, U6.8
- new net DRDY3: U5.7, U7.8
- new net INT1: U2.12, U2.16
- new net N$1: U4.12, U4.16
- new net N$11: R19.1, U5.65
- new net N$12: R32.1, U5.143
- new net N$18: R33.1, U5.138
- new net N$4: U3.12, U3.16
- new net UART7_RX: U5.58, X1.2
- new net UART7_TX: U5.59, X1.3
- new net USB_FS_DM: J1.2, U5.103
- new net USB_FS_DP: J1.3, U5.104
- new net USB_FS_OVCR: U5.92
- new net USB_FS_PWR_EN: U5.79
- net 3V3: now also J2.1, J3.4, J4.4, JP2.4, JP3.4, JP4.4, R31.2, R32.2, X1.1, X3.1; no longer LIDAR.1, OP_FLOW.1, RADIO.1, RC.1, U5.143
- net 5V: now also JP2.6, JP3.6, JP4.6, JP5.10, JP5.9
- net BOOT0: no longer U5.138
- net CSB_GYRO3: now also U5.78; no longer U5.79
- net EXTI0: now also U4.1; no longer U4.16
- net EXTI0_1: now also U2.13; no longer U2.12
- net EXTI1: now also U3.1; no longer U3.16
- net EXTI2: now also U4.13; no longer U4.12
- net EXTI3: now also U3.13; no longer U3.12
- net EXTI4: now also U2.1; no longer U2.16
- net GND: now also J1.4, J1.SH1, J1.SH2, J1.SH3, J1.SH4, J1.SH5, J1.SH6, J3.6, J3.P1, J3.P2, J3.P3, J3.P4, J3.P5, J4.1, JP2.2, JP3.2, JP4.2, JP5.3, JP5.4, R33.2, X1.6, X3.2; no longer LIDAR.6, OP_FLOW.6
- net GPIO1: now also X1.4; no longer LIDAR.4
- net I2C4_SCL: no longer LIDAR.2
- net I2C4_SDA: no longer LIDAR.3, U5.137
- net N$15: now also X3.4; no longer R19.1, U5.58
- net N$16: now also U5.66; no longer U5.59
- net N$19: now also J2.4; no longer RADIO.6, RC.6
- net NRST: now also R31.1
- net NRST_O: now also JP5.1; no longer JP1.6
- net SPI4_CS: now also J3.2
- net SPI4_MISO: now also J3.7
- net SPI4_MOSI: now also J3.3
- net SPI4_SCK: now also J3.5
- net SPI6_CS: no longer OP_FLOW.5
- net SPI6_MISO: no longer OP_FLOW.3
- net SPI6_MOSI: no longer OP_FLOW.4
- net SPI6_SCK: no longer OP_FLOW.2
- net SWCLK_O: now also JP5.6; no longer JP1.3
- net SWDIO_O: now also JP5.2; no longer JP1.5
- net SWO_O: now also JP5.5; no longer JP1.1
- net UART4_RX: now also J4.3, U5.35; no longer JP1.4, U5.103
- net UART4_TX: now also J4.2, U5.34; no longer JP1.2, U5.104
- net UART5_RX: now also X3.3, X3.6; no longer RC.3
- net UART5_TX: now also X3.5; no longer RC.2
- net UART8_RX: now also J2.3; no longer RADIO.3
- net UART8_TX: now also J2.2; no longer RADIO.2
- net XSHUT: now also X1.5; no longer LIDAR.5
Routing:
- net 5V: track 41.7 -> 188.1 mm, vias 0 -> 1
- net USB_FS_DP: track 0.00 -> 142.8 mm
- net GND: track 424.3 -> 550.0 mm, vias 16 -> 18
- net USB_FS_DM: track 0.00 -> 95.3 mm, vias 0 -> 2
- net SPI6_CS: track 128.8 -> 40.0 mm, vias 3 -> 2
- net SPI6_MISO: track 105.8 -> 25.2 mm, vias 3 -> 2
- net SPI6_SCK: track 99.8 -> 24.4 mm
- net SPI6_MOSI: track 105.8 -> 30.7 mm, vias 3 -> 2
- net SPI1_SCK: track 36.2 -> 106.6 mm
- net SPI4_CS: track 18.3 -> 86.9 mm, vias 2 -> 3
- net I2C4_SDA: track 66.0 -> 0.00 mm, vias 1 -> 0
- net UART4_RX: track 33.1 -> 95.3 mm, vias 0 -> 2
- net DRDY2: track 0.00 -> 62.0 mm, vias 0 -> 2
- net UART4_TX: track 41.1 -> 99.9 mm, vias 2 -> 4
- net SPI4_SCK: track 15.6 -> 73.3 mm, vias 0 -> 3
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