File: PCB/WIP/RedundantSensors.brd (EAGLE design)
At the start: 129.5 x 108.9 mm, 176 parts, among them J1 10118192-0001LF, J3 503182-1852, J4 JST-SH-4_SMT_V, U1 TPD4F003DQDR, U10 LIS3MDLTR, U2 BMI088, U3 BMI088, U4 BMI088, U5 STM32H743ZIT6, U6 LIS3MDLTR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

Commit message: last commit
Routing:
- net GPIO_EXTI4: track 46.3 -> 45.8 mm
Other:
- board text added: "United-Sensors UCSB"
Changed lines of the file:
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@@
 <wire x1="120.63" y1="101.27" x2="-8.89" y2="101.27" width="0" layer="20"/>
 <wire x1="-8.89" y1="101.27" x2="-8.89" y2="-7.62" width="0" layer="20"/>
+<text x="101.6" y="-3.81" size="1.778" layer="21">United-Sensors
+UCSB</text>
 </plain>
 <attributes>
@@
 <param name="mtCopper" value="0.035mm 0.035mm 0.035mm 0.035mm 0.035mm 0.035mm 0.035mm 0.035mm 0.035mm 0.035mm 0.035mm 0.035mm 0.035mm 0.035mm 0.035mm 0.035mm"/>
 <param name="mtIsolate" value="1.5mm 0.15mm 0.2mm 0.15mm 0.2mm 0.15mm 0.2mm 0.15mm 0.2mm 0.15mm 0.2mm 0.15mm 0.2mm 0.15mm 0.2mm"/>
-<param name="mdWireWire" value="6mil"/>
-<param name="mdWirePad" value="6mil"/>
+<param name="mdWireWire" value="3mil"/>
+<param name="mdWirePad" value="3mil"/>
 <param name="mdWireVia" value="6mil"/>
 <param name="mdPadPad" value="6mil"/>
@@
 <wire x1="71.4756" y1="60.96" x2="71.49" y2="60.96" width="0.1524" layer="1"/>
 <wire x1="69.1896" y1="58.3692" x2="69.1" y2="58.28" width="0.1524" layer="1"/>
-<wire x1="87.0204" y1="72.0852" x2="86.905" y2="72.065" width="0.1524" layer="1"/>
 <wire x1="88.392" y1="72.8472" x2="88.392" y2="73.3044" width="0.1524" layer="1"/>
 <wire x1="88.392" y1="73.3044" x2="88.355" y2="73.365" width="0.1524" layer="1"/>
 <wire x1="88.392" y1="72.8472" x2="88.355" y2="72.715" width="0.1524" layer="1"/>
 <wire x1="87.3252" y1="69.9516" x2="87.349" y2="69.85" width="0.1524" layer="1"/>
-<wire x1="86.868" y1="72.0852" x2="86.905" y2="72.065" width="0.1524" layer="1"/>
 <wire x1="72.39" y1="53.6448" x2="72.39" y2="53.621" width="0.1524" layer="1"/>
 <wire x1="85.6488" y1="65.9892" x2="85.67" y2="66.04" width="0.1524" layer="1"/>
@@
 <contactref element="R46" pad="1"/>
 <contactref element="JP4" pad="5"/>
-<wire x1="68.1228" y1="72.5424" x2="68.1228" y2="68.58" width="0.1524" layer="1"/>
 <wire x1="69.1896" y1="73.6092" x2="68.1228" y2="72.5424" width="0.1524" layer="1"/>
-<wire x1="68.1228" y1="68.58" x2="68" y2="68.58" width="0.1524" layer="1"/>
 <wire x1="69.1896" y1="73.6092" x2="69.16" y2="73.66" width="0.1524" layer="1"/>
 <wire x1="66.9036" y1="72.5424" x2="68.1228" y2="72.5424" width="0.1524" layer="1"/>
@@
 <wire x1="68.58" y1="92.6592" x2="67.5132" y2="91.5924" width="0.1524" layer="1"/>
 <wire x1="68.58" y1="92.6592" x2="68.58" y2="92.71" width="0.1524" layer="1"/>
+<wire x1="68" y1="68.58" x2="68" y2="72.4196" width="0.1524" layer="1"/>
+<wire x1="68" y1="72.4196" x2="68.1228" y2="72.5424" width="0.1524" layer="1"/>
 </signal>
 <signal name="SPI3_SCK">
@@
 <wire x1="67.6656" y1="48.6156" x2="65.6844" y2="48.6156" width="0.1524" layer="16"/>
 <wire x1="65.6844" y1="48.6156" x2="63.5" y2="50.8" width="0.1524" layer="16"/>
-<wire x1="63.7004" y1="55.88" x2="63.7004" y2="62.024" width="0.1524" layer="16"/>
 <wire x1="63.7004" y1="62.024" x2="73.4568" y2="71.7804" width="0.1524" layer="16"/>
 <wire x1="63.5" y1="50.8" x2="63.5" y2="53.34" width="0.1524" layer="16"/>
-<wire x1="63.5" y1="53.34" x2="64.77" y2="54.61" width="0.1524" layer="16"/>
-<wire x1="64.77" y1="54.61" x2="64.77" y2="54.8104" width="0.1524" layer="16"/>
-<wire x1="64.77" y1="54.8104" x2="63.7004" y2="55.88" width="0.1524" layer="16"/>
+<wire x1="64.1068" y1="54.86135" x2="63.7004" y2="55.26775" width="0.1524" layer="16"/>
+<wire x1="63.5" y1="53.34" x2="64.1068" y2="53.9468" width="0.1524" layer="16"/>
+<wire x1="64.1068" y1="53.9468" x2="64.1068" y2="54.86135" width="0.1524" layer="16"/>
+<wire x1="63.7004" y1="55.26775" x2="63.7004" y2="62.024" width="0.1524" layer="16"/>
 </signal>
 <signal name="GPIO_EXTI5">
@@
 </drawing>
 <compatibility>
+<note version="6.3" minversion="6.2.2" severity="warning">
+Since Version 6.2.2 text objects can contain more than one line,
+which will not be processed correctly with this version.
+</note>
 <note version="8.2" severity="warning">
 Since Version 8.2, EAGLE supports online libraries. The ids
