File: PCB/WIP/RedundantSensors.sch (EAGLE design)
At the start: 104 parts, among them J1 10118192-0001LF, U1 TPD4F003DQDR, U10 LIS3MDLTR, U2 BMI088, U3 BMI088, U4 BMI088, U5 STM32H743ZIT6, U6 LIS3MDLTR, U7 LIS3MDLTR, Y1 ECS-TXO-3225MV-400-TR, Y2 ABLS-8.000MHZ-B2-T

Commit message: rought draft #2, no issues in wiring but still under the board
Parts:
- added C53: 0.1uF, SparkFun-Capacitors:0.1UF-0603-25V-5%
- added C54: 4.7uF, SparkFun-Capacitors:4.7UF0603
- added C55, C56: 4.7pF, SparkFun-Capacitors:1.0UF-0805-25V-10%
- added JP2, JP3, JP4: (no value), pinhead:PINHD-2X3
- added L1: BLM03AG601SN1D, BLM03AG601SN1D:BLM03AG601SN1D
- added R20, R21, R22, R25, R26, R27, R28, R29: 0, SparkFun-Resistors:10KOHM-0402-1/16W-1%
- added R30: 10k, SparkFun-Resistors:10KOHM-0402-1/16W-1%
- R11: value 22 -> 0; device SparkFun-Resistors:22OHM-0402-1/10W-1% -> SparkFun-Resistors:10KOHM-0402-1/16W-1%
- Y1: value ECS-TXO-3225MV-400-TR -> 8MHz; device SamacSys_Parts:ECS-TXO-3225MV-400-TR -> ce-capstone:ABLS-8.000MHZ-B2-T
- Y2: value ABLS-8.000MHZ-B2-T -> 8MHz
Connections:
- removed net GND1: C14.2, C15.2, C16.2, C17.2, C18.2, C20.2, C21.2, C22.2
- removed net GND2: C19.2
- removed net GND3: C38.2
- removed net GND4: C39.2
- removed net N$1: R11.1, Y1.OUTPUT
- removed net VDD: C15.1, C16.1, C17.1, C18.1, C20.1, C21.1, C22.1
- removed net VREF1: C14.1
- removed net VREF2: C19.1
- removed net VREF3: C38.1
- removed net VREF4: C39.1
- new net N$21: R11.1, U4.SCL/SCK
- new net N$22: R20.1, U4.SDA/SDI
- new net N$24: R21.2, U4.SDO1
- new net N$25: R22.2, U3.SDO1
- new net N$26: R25.1, U2.SCL/SCK
- new net N$27: R26.1, U2.SDA/SDI
- new net N$28: R27.2, U2.SDO1
- new net N$29: R28.1, U3.SCL/SCK
- new net N$30: R29.1, U3.SDA/SDI
- new net OSC32_IN: C55.2, U5G$2.PC14/OSC32_IN, Y1.2
- new net OSC32_OUT: C56.2, U5G$2.PC15/OSC32_OUT, Y1.1
- net 3V3: now also C14.1, C15.1, C16.1, C17.1, C18.1, C19.1, C20.1, C21.1, C22.1, C38.1, C39.1, L1.2; no longer Y1.TRI-STATE, Y1.VDD
- net GND: now also C14.2, C15.2, C16.2, C17.2, C18.2, C19.2, C20.2, C21.2, C22.2, C38.2, C39.2, C53.2, C54.2, C55.1, C56.1; no longer Y1.GROUND
- net OSC_IN: no longer R11.2
- net SPI1_MISO: now also JP2.5, R21.1; no longer U4.SDO1
- net SPI1_MOSI: now also JP2.3, R20.2; no longer U4.SDA/SDI
- net SPI1_SCK: now also JP2.1, R11.2; no longer U4.SCL/SCK
- net SPI2_MISO: now also JP3.5, R22.1; no longer U3.SDO1
- net SPI2_MOSI: now also JP3.3, R29.2; no longer U3.SDA/SDI
- net SPI2_SCK: now also JP3.1, R28.2; no longer U3.SCL/SCK
- net SPI3_MISO: now also JP4.5, R27.1; no longer U2.SDO1
- net SPI3_MOSI: now also JP4.3, R26.2; no longer U2.SDA/SDI
- net SPI3_SCK: now also JP4.1, R25.2; no longer U2.SCL/SCK
- net VDDA: now also R30.2
- net VREFP: now also C53.1, C54.1, L1.1, R30.1
Other:
- note added: "connects to spi and can debug"
- moved on the sheet: C14, C15, C16, C17, C18, C19, C20, C21, C22, C38, C39, R11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

Commit message: snapshot before making changes suggested by phil
Parts:
- removed JP1: (no value), pinhead:PINHD-2X3
- removed LIDAR, OP_FLOW, RADIO, RC: B6B-ZR, jst:B6B-ZR
- added J2, J4: JST-SH-4_SMT_V, con-JST-SH:JST-SH-4_SMT_V
- added J3: 503182-1852, 503182-1852:503182-1852
- added JP5: (no value), jumper:JP5Q
- added R31: 10k, SparkFun-Resistors:10KOHM-0603-1/10W-1%
- added R32, R33: 1000, SparkFun-Resistors:10KOHM-0402-1/16W-1%
- added X1: LiDAR, con-jst2:06FLZ-SM1
- added X3: RC, con-jst:06FLZ-SM1
- Y1: value 8MHz -> 32MHz
Connections:
- removed net IMU_INT3: U3.INT2, U3.INT4
- removed net N$20: U4.INT2, U4.INT4
- removed net N$23: U2.INT2, U2.INT4
- new net 3.3V: JP5.7, JP5.8
- new net DRDY1: U10.DRDY, U5G$4.PG10
- new net DRDY2: U5G$2.PC4, U6.DRDY
- new net DRDY3: U5G$2.PC13, U7.DRDY
- new net INT1: U2.INT1, U2.INT3
- new net N$1: U4.INT1, U4.INT3
- new net N$11: R19.1, U5G$3.PE12
- new net N$12: R32.1, U5G$1.PDR_ON
- new net N$18: R33.1, U5G$1.BOOT0
- new net N$4: U3.INT1, U3.INT3
- new net UART7_RX: U5G$3.PE7, X1-2.1
- new net UART7_TX: U5G$3.PE8, X1-3.1
- new net USB_FS_DM: J1.D-, U5G$1.PA11
- new net USB_FS_DP: J1.D+, U5G$1.PA12
- new net USB_FS_OVCR: U5G$4.PG7
- new net USB_FS_PWR_EN: U5G$3.PD10
- net 3V3: now also J2-1.P, J3.VDD, J4-4.P, JP2.4, JP3.4, JP4.4, R31.2, R32.2, X1-1.1, X3-1.1; no longer LIDAR.1, OP_FLOW.1, RADIO.1, RC.1, U5G$1.PDR_ON
- net 5V: now also JP2.6, JP3.6, JP4.6, JP5.10, JP5.9
- net BOOT0: no longer U5G$1.BOOT0
- net CSB_GYRO3: now also U5G$3.PD9; no longer U5G$3.PD10
- net EXTI0: now also U4.INT2; no longer U4.INT1
- net EXTI0_1: now also U2.INT4; no longer U2.INT3
- net EXTI1: now also U3.INT2; no longer U3.INT1
- net EXTI2: now also U4.INT4; no longer U4.INT3
- net EXTI3: now also U3.INT4; no longer U3.INT3
- net EXTI4: now also U2.INT2; no longer U2.INT1
- net GND: now also J1.ID, J1.SHIELD, J3.SHIELD, J3.VSS, J4-1.P, JP2.2, JP3.2, JP4.2, JP5.3, JP5.4, R33.2, X1-6.1, X3-2.1; no longer LIDAR.6, OP_FLOW.6
- net GPIO1: now also X1-4.1; no longer LIDAR.4
- net I2C4_SCL: no longer LIDAR.2
- net I2C4_SDA: no longer LIDAR.3, U5G$2.PB7
- net N$15: now also X3-4.1; no longer R19.1, U5G$3.PE7
- net N$16: now also U5G$3.PE13; no longer U5G$3.PE8
- net N$19: now also J2-4.P; no longer RADIO.6, RC.6
- net NRST: now also R31.1
- net NRST_O: now also JP5.1; no longer JP1.6
- net SPI4_CS: now also J3.CD/DAT3
- net SPI4_MISO: now also J3.DAT0
- net SPI4_MOSI: now also J3.CMD
- net SPI4_SCK: now also J3.CLK
- net SPI6_CS: no longer OP_FLOW.5
- net SPI6_MISO: no longer OP_FLOW.3
- net SPI6_MOSI: no longer OP_FLOW.4
- net SPI6_SCK: no longer OP_FLOW.2
- net SWCLK_O: now also JP5.6; no longer JP1.3
- net SWDIO_O: now also JP5.2; no longer JP1.5
- net SWO_O: now also JP5.5; no longer JP1.1
- net UART4_RX: now also J4-3.P, U5G$1.PA1; no longer JP1.4, U5G$1.PA11
- net UART4_TX: now also J4-2.P, U5G$1.PA0; no longer JP1.2, U5G$1.PA12
- net UART5_RX: now also X3-3.1, X3-6.1; no longer RC.3
- net UART5_TX: now also X3-5.1; no longer RC.2
- net UART8_RX: now also J2-3.P; no longer RADIO.3
- net UART8_TX: now also J2-2.P; no longer RADIO.2
- net XSHUT: now also X1-5.1; no longer LIDAR.5
Other:
- note added: "OP_Flow"
- note added: "SD Card"
- note added: "Telemetry"
- moved on the sheet: C23, C36, C41, C42, C43, C44, C45, C46, C47, C48, C6, C7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

Commit message: PCB updated
Parts:
- removed C55, C56: 4.7pF, SparkFun-Capacitors:1.0UF-0805-25V-10%
- removed J2: JST-SH-4_SMT_V, con-JST-SH:JST-SH-4_SMT_V
- removed R19, R8, R9: RT0402FRE07220RL, ce-capstone:RT0402FRE07220RL
- removed S1, S2: LL3301FF065QJ, ce-capstone:LL3301FF065QJ
- removed Y1: 32MHz, ce-capstone:ABLS-8.000MHZ-B2-T
- added C57, C58: 0.1uF, SparkFun-Capacitors:0.1UF-0603-25V-5%
- added C59, C60: 1.0uF, SparkFun-Capacitors:1.0UF-0402-16V-10%
- added FL4, FL5, FL6: BLM03AG601SN1D, BLM03AG601SN1D:BLM03AG601SN1D
- added L6, L8: 150uH, inductors:MICC10
- added LD1: PL006-WCR12, led:PL006-WCR12
- added LD2: PL006-WCG13, led:PL006-WCR12
- added LD3: PL006-WCY01, led:PL006-WCR12
- added R34, R35, R36, R39, R40, R41, R42, R43, R44, R45, R46, R47, R48, R49, R50, R51, R52, R54, R55, R56, R57, R58, R59, R76, R77: 22, SparkFun-Resistors:10KOHM-0402-1/16W-1%
- added R37, R38, R64, R65, R67, R68: 47k, SparkFun-Resistors:10KOHM-0402-1/16W-1%
- added R53, R63, R75, R78, R79, R80, R81: 10K, ce-capstone:RT0402FRE07220RL
- added R60, R61, R62: 22, SparkFun-Resistors:22OHM-0402-1/10W-1%
- added R69, R70, R71: 270, ce-capstone:RT0402FRE07220RL
- added T1, T2, T3: (no value), transistor:MUN2213T1-NPN_DRIVER-SC59-BEC
- added X2: Telemetry, con-jst:06FLZ-SM1
- R31, R5: value 10k -> 22; device SparkFun-Resistors:10KOHM-0603-1/10W-1% -> SparkFun-Resistors:10KOHM-0402-1/16W-1%
- R6, R7: value RT0402FRE07220RL -> 10K
Connections:
- removed net BOOT0: R5.1, S1.3, S1.4
- removed net DRDY1: U10.DRDY, U5G$4.PG10
- removed net DRDY2: U5G$2.PC4, U6.DRDY
- removed net DRDY3: U5G$2.PC13, U7.DRDY
- removed net EXTI1: R24.2, U3.INT2
- removed net EXTI3: R17.2, U3.INT4
- removed net EXTI4: R18.2, U2.INT2
- removed net GPIO_EXTI00: R23.1, U5G$4.PG0
- removed net INT1: U2.INT1, U2.INT3
- removed net JTRST: U5G$2.PB4(!JTRST!)
- removed net N$1: U4.INT1, U4.INT3
- removed net N$10: C33.2, FL3.1, U3.VDDIO
- removed net N$19: J2-4.P
- removed net N$4: U3.INT1, U3.INT3
- removed net N$8: C27.2, FL2.1, U4.VDDIO
- removed net N$9: C30.2, FL1.1, U2.VDDIO
- removed net OSC32_IN: C55.2, U5G$2.PC14/OSC32_IN, Y1.2
- removed net OSC32_OUT: C56.2, U5G$2.PC15/OSC32_OUT, Y1.1
- new net CSB_ACCEL4: R6.2, U4.CSB1
- new net DM: C59.2, J1.D-, L8.1
- new net DP: C59.1, J1.D+, L6.1
- new net DRDY1_ACC: U4.INT1, U5G$3.PD11
- new net DRDY1_ACC2: U2.INT1, U5G$4.PF13
- new net DRDY1_ACC3: U3.INT1, U5G$4.PG2
- new net DRDY2_GYRO: U2.INT3, U4.INT3, U5G$3.PE10
- new net DRDY2_GYRO2: U5G$4.PF14
- new net DRDY2_GYRO3: U3.INT3, U5G$4.PG3
- new net EXTI0_2: R23.2, U3.INT2
- new net EXTI2_1: R18.2, U2.INT4
- new net EXTI2_2: R24.2, U3.INT4
- new net GPIO_EXTI10: R24.1, U5G$2.PB10
- new net GPIO_EXTI11: R61.2, U5G$4.PF11
- new net GPIO_EXTI12: R62.2, U5G$4.PF12
- new net GPIO_EXTI5: R18.1, U5G$4.PG5
- new net GPIO_EXTI6: R23.1, U5G$4.PG6
- new net LED01: T2.B, U5G$1.PA4
- new net LED02: T1.B, U5G$2.PC5
- new net LED03: T3.B, U5G$2.PC6
- new net N$20: R5.1, U5G$1.PA1
- new net N$23: R40.2, U5G$2.PC2_C
- new net N$31: R34.1, U5G$3.PD6
- new net N$32: R35.1, U5G$3.PD5
- new net N$33: R36.1, U5G$1.PA5
- new net N$36: R39.1, U5G$2.PB13
- new net N$37: R41.2, U5G$2.PC3_C
- new net N$38: R31.1, U5G$3.PD1
- new net N$39: R42.1, U5G$2.PB5
- new net N$40: R43.1, U5G$2.PB6
- new net N$41: R44.2, U5G$2.PC10
- new net N$42: R45.2, U5G$2.PC11
- new net N$43: R46.2, U5G$2.PC12
- new net N$44: R47.2, U5G$4.PG12
- new net N$45: R48.2, U5G$4.PG13
- new net N$46: R49.2, U5G$4.PG14
- new net N$47: R50.1, U5G$4.PF7
- new net N$48: R51.1, U5G$4.PF8
- new net N$49: R52.1, U5G$4.PF9
- new net N$50: R57.2, U5G$3.PE6
- new net N$51: R58.2, U5G$3.PE1
- new net N$52: R59.2, U5G$3.PE0
- new net N$53: C43.2, C44.2, C45.2, FL5.1, U6.VDD
- new net N$54: C58.2, U7.C1
- new net N$55: C46.2, C47.2, C48.2, FL6.1, U7.VDD
- new net N$56: R60.1, U10.INT
- new net N$57: R61.1, U6.INT
- new net N$58: R62.1, U7.INT
- new net N$59: LD2.C, T2.C
- new net N$60: LD2.A, R69.1
- new net N$61: LD1.C, T1.C
- new net N$62: LD1.A, R70.1
- new net N$63: LD3.C, T3.C
- new net N$64: LD3.A, R71.1
- new net N$67: R54.2, U5G$3.PE2
- new net N$68: R76.1, U5G$3.PD7
- new net N$69: R77.2, U5G$4.PG9
- new net SDMCC_CK: J3.CLK, R64.1, U5G$2.PC1
- new net SDMCC_CMD: J3.CMD, R38.1, U5G$1.PA0
- new net SDMCC_D0: J3.DAT0, R67.1, U5G$2.PB14
- new net SDMCC_D1: J3.DAT1, R65.1, U5G$2.PB15
- new net SDMCC_D2: J3.DATA2, R68.1, U5G$4.PG11
- new net SDMCC_D3: J3.CD/DAT3, R37.1, U5G$2.PB4(!JTRST!)
- new net TIM1_CH1: U5G$3.PE9
- new net TIM1_CH2: U5G$3.PE11
- new net TIM1_CH3: U5G$3.PE13
- new net TIM1_CH4: U5G$3.PE14
- new net TIM3_CH1: U5G$1.PA6
- new net TIM3_CH2: U5G$1.PA7
- new net TIM3_CH3: U5G$2.PB0
- new net TIM3_CH4: U5G$2.PB1
- new net TIM4_CH2: U5G$2.PB7, X3-3.1
- new net UART8_CTS: U5G$3.PD14, X2-2.1
- new net UART8_RTS: U5G$3.PD15, X2-3.1
- new net USART1_RX: U5G$1.PA10
- new net USART1_TX: U5G$1.PA9
- net 3V3: now also C27.2, C30.2, C33.2, FL1.1, FL2.1, FL3.1, FL4.2, FL5.2, FL6.2, R37.2, R38.2, R53.1, R6.1, R63.1, R64.2, R65.2, R67.2, R68.2, R69.2, R7.1, R70.2, R71.2, R75.1, R78.1, R79.1, R80.1, R81.1, U2.VDDIO, U3.VDDIO, U4.VDDIO; no longer C36.2, C41.2, C42.2, C43.2, C44.2, C45.2, C46.2, C47.2, C48.2, J2-1.P, R31.2, S1.1, S1.2, U10.VDD, U6.VDD, U7.VDD
- net 5V_IN: now also X2-1.1
- net CSB_ACCEL1: now also U5G$3.PE12; no longer R19.2, U4.CSB1
- net CSB_ACCEL2: now also R75.2, U5G$3.PE15; no longer R9.2
- net CSB_ACCEL3: now also R53.2, U5G$3.PD8; no longer R6.1
- net CSB_GYRO1: now also R63.2, U5G$4.PF15; no longer R8.2
- net CSB_GYRO2: now also R78.2, U5G$3.PD3; no longer R7.1
- net CSB_GYRO3: now also R7.2
- net EXTI0_1: now also R17.2, U2.INT2; no longer R23.2, U2.INT4
- net GND: now also C23.1, C57.1, C58.1, T1.E, T2.E, T3.E, X2-6.1; no longer C23.2, C55.1, C56.1, R5.2, S2.3, S2.4, U10.C1, U6.C1, U7.C1
- net GPIO_EXTI0: now also U5G$4.PG0; no longer U5G$3.PD0
- net GPIO_EXTI1: no longer R24.1, U5G$3.PD1
- net GPIO_EXTI2: now also U5G$4.PF2; no longer U5G$3.PD2
- net GPIO_EXTI3: now also R60.2, U5G$4.PF3; no longer R17.1, U5G$3.PD3
- net GPIO_EXTI4: now also R17.1, U5G$4.PG4; no longer R18.1, U5G$3.PD4
- net N$11: now also C23.2, U10.C1; no longer R19.1, U5G$3.PE12
- net N$13: now also R55.2, U5G$3.PE4; no longer R6.2, U5G$3.PD7
- net N$14: now also R56.2, U5G$3.PE5; no longer R7.2, U5G$3.PD6
- net N$16: now also C36.2, C41.2, C42.2, FL4.1, U10.VDD; no longer R8.1, U5G$3.PE13
- net N$17: now also C57.2, U6.C1; no longer R9.1, U5G$3.PE9
- net NRST: no longer C23.1, R31.1, S2.1, S2.2
- net SPI1_MISO: now also JP2.3, R77.1, U4.SDO2; no longer JP2.5, U5G$1.PA6
- net SPI1_MOSI: now also JP2.5, R76.2; no longer JP2.3, U5G$1.PA7
- net SPI1_SCK: now also R36.2; no longer U5G$1.PA5
- net SPI2_MISO: now also JP3.3, R40.1, U3.SDO2; no longer JP3.5, U5G$2.PB14
- net SPI2_MOSI: now also JP3.5, R41.1; no longer JP3.3, U5G$2.PB15
- net SPI2_SCK: now also R39.2; no longer U5G$2.PB13
- net SPI3_MISO: now also JP4.3, R45.1, U2.SDO2; no longer JP4.5, U5G$2.PC11
- net SPI3_MOSI: now also JP4.5, R46.1; no longer JP4.3, U5G$2.PC12
- net SPI3_SCK: now also R44.1; no longer U5G$2.PC10
- net SPI4_CS: now also R55.1, R81.2; no longer J3.CD/DAT3, U5G$3.PE4
- net SPI4_MISO: now also R56.1, U7.SDO/SA1; no longer J3.DAT0, U5G$3.PE5, U7.SDA/SDI/SDO
- net SPI4_MOSI: now also R57.1, U7.SDA/SDI/SDO; no longer J3.CMD, U5G$3.PE6, U7.SDO/SA1
- net SPI4_SCK: now also R54.1; no longer J3.CLK, U5G$3.PE2
- net SPI5_CS: now also R80.2
- net SPI5_MISO: now also R51.2, U6.SDO/SA1; no longer U5G$4.PF8, U6.SDA/SDI/SDO
- net SPI5_MOSI: now also R52.2, U6.SDA/SDI/SDO; no longer U5G$4.PF9, U6.SDO/SA1
- net SPI5_SCK: now also R50.2; no longer U5G$4.PF7
- net SPI6_CS: now also R79.2
- net SPI6_MISO: now also R47.1, U10.SDO/SA1; no longer U10.SDA/SDI/SDO, U5G$4.PG12
- net SPI6_MOSI: now also R49.1, U10.SDA/SDI/SDO; no longer U10.SDO/SA1, U5G$4.PG14
- net SPI6_SCK: now also R48.1; no longer U5G$4.PG13
- net UART4_RX: now also R5.2, X3-6.1; no longer J4-3.P, U5G$1.PA1
- net UART4_TX: now also R31.2, X3-5.1; no longer J4-2.P, U5G$1.PA0
- net UART5_RX: now also J4-3.P, R42.2; no longer U5G$2.PB5, X3-3.1, X3-6.1
- net UART5_TX: now also J4-2.P, R43.2; no longer U5G$2.PB6, X3-5.1
- net UART8_RX: now also R59.1, X2-4.1; no longer J2-3.P, U5G$3.PE0
- net UART8_TX: now also R58.1, X2-5.1; no longer J2-2.P, U5G$3.PE1
- net USART2_RX: now also R34.2
- net USART2_TX: now also R35.2
- net USB_FS_DM: now also C60.2, L8.2; no longer J1.D-
- net USB_FS_DP: now also C60.1, L6.2; no longer J1.D+
- net XSHUT: now also U5G$2.PC7; no longer U5G$2.PC1
Other:
- note added: "LED for ardupilot"
- note added: "green"
- note added: "red"
- note added: "yellow"
- note removed: "Buttons"
- note removed: "Reset"
- note removed: "Telemetry"
- note removed: "User"
- moved on the sheet: C23, J3, R11, R17, R18, R20, R23, R24, R31, R6, R7, U5G$3
