File: PCB/WIP/RedundantSensors.sch (EAGLE design)
At the start: 176 parts, among them J1 10118192-0001LF, J3 503182-1852, J4 JST-SH-4_SMT_V, U1 TPD4F003DQDR, U10 LIS3MDLTR, U2 BMI088, U3 BMI088, U4 BMI088, U5 STM32H743ZIT6, U6 LIS3MDLTR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

Commit message: PCB prelim
Connections:
- net DRDY1_ACC2: now also U5G$3.PD0; no longer U5G$4.PF13
- net DRDY2_GYRO: now also U5G$1.PA15(JTDI); no longer U5G$3.PE10
Changed lines of the file:
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@@
 <net name="DRDY2_GYRO" class="0">
-<segment>
-<pinref part="U5" gate="G$3" pin="PE10"/>
-<wire x1="-35.56" y1="185.42" x2="-17.78" y2="185.42" width="0.1524" layer="91"/>
-<label x="-22.86" y="185.42" size="1.778" layer="95"/>
-</segment>
 <segment>
 <pinref part="U4" gate="G$1" pin="INT3"/>
@@
 <label x="363.22" y="63.5" size="1.778" layer="95"/>
 </segment>
+<segment>
+<wire x1="-48.26" y1="243.84" x2="-66.04" y2="243.84" width="0.1524" layer="91"/>
+<label x="-48.26" y="243.84" size="1.778" layer="95" rot="R180"/>
+<pinref part="U5" gate="G$1" pin="PA15(JTDI)"/>
+</segment>
 </net>
 <net name="DRDY1_ACC2" class="0">
-<segment>
-<pinref part="U5" gate="G$4" pin="PF13"/>
-<wire x1="33.02" y1="180.34" x2="15.24" y2="180.34" width="0.1524" layer="91"/>
-<label x="10.16" y="180.34" size="1.778" layer="95"/>
-</segment>
 <segment>
 <pinref part="U2" gate="G$1" pin="INT1"/>
@@
 <label x="363.22" y="68.58" size="1.778" layer="95"/>
 </segment>
+<segment>
+<wire x1="-71.12" y1="210.82" x2="-88.9" y2="210.82" width="0.1524" layer="91"/>
+<label x="-93.98" y="210.82" size="1.778" layer="95"/>
+<pinref part="U5" gate="G$3" pin="PD0"/>
+</segment>
 </net>
